Commit message: fix

File: arms_moveit_config/config/cl_arms.ros2_control.xacro (robot description, xacro)
@@ -1,10 +1,10 @@
 <?xml version="1.0"?>
 <robot xmlns:xacro="http://www.ros.org/wiki/xacro">
-    <xacro:macro name="cl_arms_ros2_control" params="name initial_positions_file">
+    <xacro:macro name="cl_arms_ros2_control" params="name initial_positions_file plugin_name">
         <xacro:property name="initial_positions" value="${xacro.load_yaml(initial_positions_file)['initial_positions']}"/>
         <ros2_control name="${name}" type="system">
             <hardware>
                 <!-- By default, set up controllers for simulation. This won't work on real hardware -->
-                <plugin>mock_components/GenericSystem</plugin>
+                <plugin>${plugin_name}</plugin>
             </hardware>
             <joint name="R_SHOULDER_P">

File: arms_moveit_config/config/cl_arms.urdf.xacro (robot description, xacro)
@@ -6,4 +6,7 @@
     <!-- Import control_xacro -->
     <xacro:include filename="cl_arms.ros2_control.xacro" />
-    <xacro:cl_arms_ros2_control name="FakeSystem" initial_positions_file="$(arg initial_positions_file)"/>
+    <xacro:cl_arms_ros2_control
+    name="FakeSystem"
+    initial_positions_file="$(arg initial_positions_file)"
+    plugin_name = "annin_ar4_driver/ARHardwareInterface" />
 </robot>
